Commit message: Update r2d2.urdf.xacro

File: src/my_r2d2/urdf/r2d2.urdf.xacro (robot description, xacro)
@@ -213,8 +213,8 @@
     <origin xyz="${.707*width+0.04} 0 ${.707*width}"/>
   </joint>
-	<link name="lense">
-    <visual>
-      <geometry>
-				<cylinder radius="0.035" length="0.001"/>
+<link name="lense">
+    <visual>
+      <geometry>
+	<cylinder radius="0.035" length="0.001"/>
       </geometry>
       <material name="black"/>

Commit message: Third homework done

File: src/my_r2d2/urdf/r2d2.urdf.xacro (robot description, xacro)
@@ -8,4 +8,5 @@
   <xacro:property name="wheeldiam" value="0.07" />
   <xacro:property name="pi" value="3.1415" />
+  <xacro:property name="footprintlen" value="0.17" />
   <material name="blue">
     <color rgba="0 0 0.8 1"/>
@@ -233,3 +234,9 @@
     <origin xyz="0 0 0"/>
   </joint>
+  <link name="base_footprint" />
+  <joint name="base_footprint_base_link_joint" type="fixed">
+    <parent link="base_footprint"/>
+    <child link="base_link"/>
+    <origin xyz="0 0 ${leglen/2 + wheeldiam + 0.1}"/>
+  </joint>
 </robot>
