Commit message: Small changes in homework

File: src/my_r2d2/urdf/r2d2.urdf (robot description, URDF)
Before this commit: robot myfirst, 16 links, 15 joints
Links:
- removed link left_back_wheel
- removed link left_base
- removed link left_front_wheel
- removed link left_gripper
- removed link left_leg
- removed link left_tip
- removed link right_back_wheel
- removed link right_base
- removed link right_front_wheel
- removed link right_gripper
- removed link right_leg
- removed link right_tip
- added link base_footprint
- added link eye
- added link lens; collision cylinder length=0.01 radius=${lensdiam/2}; visual cylinder length=0.01 radius=${lensdiam/2}
- link base_link: mass 10 -> None; geometry collision cylinder length=${bodylen} radius=${width}; visual cylinder length=${bodylen} radius=${width}
- link box: mass 1 -> None
- link gripper_pole: mass 0.05 -> None; geometry collision cylinder length=${polelen} radius=0.01; visual cylinder length=${polelen} radius=0.01
- link head: mass 2 -> None; geometry collision sphere radius=${width}; visual sphere radius=${width}
Joints:
- removed joint base_to_left_leg
- removed joint base_to_right_leg
- removed joint left_back_wheel_joint
- removed joint left_base_joint
- removed joint left_front_wheel_joint
- removed joint left_gripper_joint
- removed joint left_tip_joint
- removed joint right_back_wheel_joint
- removed joint right_base_joint
- removed joint right_front_wheel_joint
- removed joint right_gripper_joint
- removed joint right_tip_joint
- added joint base_footprint_base_link_joint: type fixed, parent base_footprint, child base_link, origin xyz=0 0 ${leglen/2 + wheeldiam + 0.1}
- added joint box_lens_joint: type fixed, parent box, child lens, origin xyz=0 0 0 rpy=${3*pi/2} ${2*pi} ${3*pi/2}
- added joint lens_eye_joint: type fixed, parent lens, child eye, origin xyz=0 0 0 rpy=0 0 0
- joint gripper_extension: limit lower=-0.38 upper=0 effort=1000.0 velocity=0.5 -> lower=-${width*2-.02} upper=0 effort=1000.0 velocity=0.5; origin xyz=0.19 0 0.2 rpy=0 0 0 -> xyz=${width-.01} 0 0.2 rpy=0 0 0
- joint head_swivel: origin xyz=0 0 0.3 -> xyz=0 0 ${bodylen/2}
- joint tobox: origin xyz=0.1814 0 0.1414 -> xyz=${.707*width+0.04} 0 ${.707*width}

Commit message: Third homework done

File: src/my_r2d2/urdf/r2d2.urdf (robot description, URDF)
Before this commit: robot macroed, 7 links, 6 joints
Links:
- removed link eye
Joints:
- removed joint box_lens_joint
- removed joint lens_eye_joint
- added joint box_lens_connect: type fixed, parent box, child lens, origin xyz=0 0 0 rpy=0 ${pi/2} 0
