Commit message: 4 homework done

File: src/my_r2d2/urdf/r2d2.xacro (robot description, xacro)
@@ -231,4 +231,15 @@
     <xacro:default_inertial mass="0.02"/>
   </link>
+  <joint name="box_lens_joint" type="fixed">
+    <parent link="box"/>
+    <child link="lens"/>
+    <origin xyz="0 0 0" rpy="${3*pi/2} ${2*pi} ${3*pi/2}"/>
+  </joint>
+  <link name="eye"/>
+  <joint name="lens_eye_joint" type="fixed">
+    <parent link="lens"/>
+    <child link="eye"/>
+    <origin xyz="0 0 0" rpy="0 0 0"/>
+  </joint>
   <joint name="tobox" type="fixed">
     <parent link="head"/>
@@ -236,8 +247,3 @@
     <origin xyz="${.707*width+0.04} 0 ${.707*width}"/>
   </joint>
-  <joint name="box_lens_connect" type="fixed">
-    <parent link="box"/>
-    <child link="lens"/>
-    <origin xyz="0 0 0" rpy="0 ${pi/2} 0"/>
-  </joint>
 </robot>

Commit message: Changed two files for 4 homework

File: src/my_r2d2/urdf/r2d2.xacro (robot description, xacro)
@@ -6,7 +6,5 @@
   <xacro:property name="bodylen" value="0.6" />
   <xacro:property name="baselen" value="0.4" />
-  <xacro:property name="footprintlen" value="0.17" />
   <xacro:property name="wheeldiam" value="0.07" />
-  <xacro:property name="lensdiam" value="0.07" />
   <xacro:property name="pi" value="3.1415" />
   <material name="blue">
@@ -25,4 +23,10 @@
     </inertial>
   </xacro:macro>
+  <xacro:macro name="inertial_3" params="mass ixx iyy izz">
+    <inertial>
+      <mass value="${mass}" />
+      <inertia ixx="${ixx}" ixy="0.0" ixz="0.0" iyy="${iyy}" iyz="0.0" izz="${izz}" />
+    </inertial>
+  </xacro:macro>
   <link name="base_link">
     <visual>
@@ -37,11 +41,11 @@
       </geometry>
     </collision>
-    <xacro:default_inertial mass="10"/>
+    <xacro:inertial_3 mass="10" ixx="0.4" iyy="0.4" izz="0.2"/>
   </link>
   <link name="base_footprint" />
-  <joint name="base_footprint_base_link_joint" type="fixed">
+  <joint name="base_footprint_to_base_link" type="fixed">
     <parent link="base_footprint"/>
     <child link="base_link"/>
-    <origin xyz="0 0 ${leglen/2 + wheeldiam + 0.1}"/>
+    <origin xyz="0 0 ${baselen + wheeldiam}" rpy="0 0 0"/>
   </joint>
   <xacro:macro name="wheel" params="prefix suffix reflect">
@@ -213,33 +217,7 @@
         <box size="0.08 0.08 0.08"/>
       </geometry>
-      <origin xyz="-0.04 0 0"/>
     </collision>
     <xacro:default_inertial mass="1"/>
   </link>
-  <link name="lens">
-    <visual>
-      <geometry>
-        <cylinder length="0.01" radius="${lensdiam/2}"/>
-      </geometry>
-      <material name="black"/>
-    </visual>
-    <collision>
-      <geometry>
-        <cylinder length="0.01" radius="${lensdiam/2}"/>
-      </geometry>
-    </collision>
-    <xacro:default_inertial mass="0.02"/>
-  </link>
-  <joint name="box_lens_joint" type="fixed">
-    <parent link="box"/>
-    <child link="lens"/>
-    <origin xyz="0 0 0" rpy="${3*pi/2} ${2*pi} ${3*pi/2}"/>
-  </joint>
-  <link name="eye"/>
-  <joint name="lens_eye_joint" type="fixed">
-    <parent link="lens"/>
-    <child link="eye"/>
-    <origin xyz="0 0 0" rpy="0 0 0"/>
-  </joint>
   <joint name="tobox" type="fixed">
     <parent link="head"/>
@@ -247,3 +225,29 @@
     <origin xyz="${.707*width+0.04} 0 ${.707*width}"/>
   </joint>
+  <link name="lense">
+    <visual>
+      <geometry>
+        <cylinder radius="0.03" length="0.02"/>
+      </geometry>
+      <material name="black"/>
+      <origin xyz="-0.04 0 0" rpy="0 ${pi/2} 0"/>
+    </visual>
+    <collision>
+      <geometry>
+        <cylinder radius="0.03" length="0.02"/>
+      </geometry>
+    </collision>
+    <xacro:default_inertial mass="0.1"/>
+  </link>
+  <joint name="tolense" type="fixed">
+    <parent link="box"/>
+    <child link="lense"/>
+    <origin xyz="0.05 0 0"/>
+  </joint>
+  <link name="eye"/>
+  <joint name="lensetoeye" type="fixed">
+    <parent link="lense" />
+    <child link="eye" />
+    <origin xyz="0 0 0" rpy="-1.57 0 -1.57"/>
+  </joint>
 </robot>
